File: das keyboard/das keyboard.kicad_pcb (KiCad board)
At the start: 2 copper layers, 13 parts

Commit message: updates to the pcb
Parts:
- removed KP_8, KP_9: SW_SPST, Button_Switch_Keyboard:SW_Cherry_MX_1.00u_PCB
- added +=1: SW_SPST, Button_Switch_Keyboard:SW_Cherry_MX_1.00u_PCB, B.Cu at (361.5, 56.5)
- added 1_1: SW_SPST, Button_Switch_Keyboard:SW_Cherry_MX_1.00u_PCB, B.Cu at (801.5, 56.5)
- added 2_1: SW_SPST, Button_Switch_Keyboard:SW_Cherry_MX_1.00u_PCB, B.Cu at (761.5, 56.5)
- added 3_1: SW_SPST, Button_Switch_Keyboard:SW_Cherry_MX_1.00u_PCB, B.Cu at (721.5, 56.5)
- added 4_1: SW_SPST, Button_Switch_Keyboard:SW_Cherry_MX_1.00u_PCB, B.Cu at (681.5, 56.5)
- added 5_1: SW_SPST, Button_Switch_Keyboard:SW_Cherry_MX_1.00u_PCB, B.Cu at (641.5, 56.5)
- added 6_1: SW_SPST, Button_Switch_Keyboard:SW_Cherry_MX_1.00u_PCB, B.Cu at (601.5, 56.5)
- added 7_1: SW_SPST, Button_Switch_Keyboard:SW_Cherry_MX_1.00u_PCB, B.Cu at (561.5, 56.5)
- added 8_1: SW_SPST, Button_Switch_Keyboard:SW_Cherry_MX_1.00u_PCB, B.Cu at (521.5, 56.5)
- added 9_1: SW_SPST, Button_Switch_Keyboard:SW_Cherry_MX_1.00u_PCB, B.Cu at (481.5, 56.5)
- added APPS1: SW_SPST, Button_Switch_Keyboard:SW_Cherry_MX_1.00u_PCB, B.Cu at (361.5, 221.6)
- added A_1: SW_SPST, Button_Switch_Keyboard:SW_Cherry_MX_1.00u_PCB, B.Cu at (801.9, 136.5)
- added Apostrophe_1: SW_SPST, Button_Switch_Keyboard:SW_Cherry_MX_1.00u_PCB, B.Cu at (441.5, 136.5)
- added B_1: SW_SPST, Button_Switch_Keyboard:SW_Cherry_MX_1.00u_PCB, B.Cu at (641.5, 176.5)
- added Backslash1: SW_SPST, Button_Switch_Keyboard:SW_Cherry_MX_1.50u_PCB, B.Cu at (321.5, 95.9)
- added Backspace1: SW_SPST, Button_Switch_Keyboard:SW_Cherry_MX_2.00u_PCB, B.Cu at (321.5, 56.5)
- added CAPS_1: SW_SPST, Button_Switch_Keyboard:SW_Cherry_MX_1.50u_PCB, B.Cu at (841.5, 136.5)
- added C_1: SW_SPST, Button_Switch_Keyboard:SW_Cherry_MX_1.00u_PCB, B.Cu at (721.5, 176.5)
- added Close_Bracket1: SW_SPST, Button_Switch_Keyboard:SW_Cherry_MX_1.00u_PCB, B.Cu at (361.5, 96.5)
- added D10: 1N4001, Diode_THT:D_DO-41_SOD81_P10.16mm_Horizontal, B.Cu at (41.5, 116.5)
- added D100: 1N4001, Diode_THT:D_DO-41_SOD81_P10.16mm_Horizontal, B.Cu at (801.9, 195.4)
- added D101: 1N4001, Diode_THT:D_DO-41_SOD81_P10.16mm_Horizontal, B.Cu at (871.5, 136.5)
- added D102: 1N4001, Diode_THT:D_DO-41_SOD81_P10.16mm_Horizontal, B.Cu at (871.5, 166.5)
- added D103: 1N4001, Diode_THT:D_DO-41_SOD81_P10.16mm_Horizontal, B.Cu at (799.4, 213.2)
- added D104: 1N4001, Diode_THT:D_DO-41_SOD81_P10.16mm_Horizontal, B.Cu at (841.5, 126.5)
- added D105: 1N4001, Diode_THT:D_DO-41_SOD81_P10.16mm_Horizontal, B.Cu at (850.2, -0.18)
- added D106: 1N4001, Diode_THT:D_DO-41_SOD81_P10.16mm_Horizontal, B.Cu at (851.5, 76.5)
- added D107: 1N4001, Diode_THT:D_DO-41_SOD81_P10.16mm_Horizontal, B.Cu at (851.5, 116.5)
- added D108: 1N4001, Diode_THT:D_DO-41_SOD81_P10.16mm_Horizontal, B.Cu at (841.5, 211.6)
- added D11: 1N4001, Diode_THT:D_DO-41_SOD81_P10.16mm_Horizontal, B.Cu at (57.7, 137.0)
- added D12: 1N4001, Diode_THT:D_DO-41_SOD81_P10.16mm_Horizontal, B.Cu at (41.5, 196.5)
- added D13: 1N4001, Diode_THT:D_DO-41_SOD81_P10.16mm_Horizontal, B.Cu at (81.5, 45.5)
- added D14: 1N4001, Diode_THT:D_DO-41_SOD81_P10.16mm_Horizontal, B.Cu at (81.5, 116.5)
- added D15: 1N4001, Diode_THT:D_DO-41_SOD81_P10.16mm_Horizontal, B.Cu at (65.3, 137.0)
- added D16: 1N4001, Diode_THT:D_DO-41_SOD81_P10.16mm_Horizontal, B.Cu at (80.5, 205.6)
- added D17: 1N4001, Diode_THT:D_DO-41_SOD81_P10.16mm_Horizontal, B.Cu at (57.7, 243.7)
- added D18: 1N4001, Diode_THT:D_DO-41_SOD81_P10.16mm_Horizontal, B.Cu at (171.5, 126.5)
- added D19: 1N4001, Diode_THT:D_DO-41_SOD81_P10.16mm_Horizontal, B.Cu at (161.5, 76.5)
- added D20: 1N4001, Diode_THT:D_DO-41_SOD81_P10.16mm_Horizontal, B.Cu at (161.8, 142.1)
- added D21: 1N4001, Diode_THT:D_DO-41_SOD81_P10.16mm_Horizontal, B.Cu at (171.5, -3.50)
- added D22: 1N4001, Diode_THT:D_DO-41_SOD81_P10.16mm_Horizontal, B.Cu at (251.5, 206.5)
- added D23: 1N4001, Diode_THT:D_DO-41_SOD81_P10.16mm_Horizontal, B.Cu at (202.5, 76.0)
- added D24: 1N4001, Diode_THT:D_DO-41_SOD81_P10.16mm_Horizontal, B.Cu at (201.5, 116.5)
- added D25: 1N4001, Diode_THT:D_DO-41_SOD81_P10.16mm_Horizontal, B.Cu at (100.9, 253.8)
- added D26: 1N4001, Diode_THT:D_DO-41_SOD81_P10.16mm_Horizontal, B.Cu at (601.5, 6.50)
- added D27: 1N4001, Diode_THT:D_DO-41_SOD81_P10.16mm_Horizontal, B.Cu at (207.5, 251.6)
- added D28: 1N4001, Diode_THT:D_DO-41_SOD81_P10.16mm_Horizontal, B.Cu at (241.5, 76.5)
- added D29: 1N4001, Diode_THT:D_DO-41_SOD81_P10.16mm_Horizontal, B.Cu at (227.9, 96.3)
- added D30: 1N4001, Diode_THT:D_DO-41_SOD81_P10.16mm_Horizontal, B.Cu at (251.5, -3.50)
- added D31: 1N4001, Diode_THT:D_DO-41_SOD81_P10.16mm_Horizontal, B.Cu at (166.9, 241.1)
- added D32: 1N4001, Diode_THT:D_DO-41_SOD81_P10.16mm_Horizontal, B.Cu at (321.5, -5.26)
- added D33: 1N4001, Diode_THT:D_DO-41_SOD81_P10.16mm_Horizontal, B.Cu at (321.8, 215.7)
- added D34: 1N4001, Diode_THT:D_DO-41_SOD81_P10.16mm_Horizontal, B.Cu at (520.0, 35.4)
- added D35: 1N4001, Diode_THT:D_DO-41_SOD81_P10.16mm_Horizontal, B.Cu at (631.7, 144.6)
- added D36: 1N4001, Diode_THT:D_DO-41_SOD81_P10.16mm_Horizontal, B.Cu at (401.5, 1.42)
- added D37: 1N4001, Diode_THT:D_DO-41_SOD81_P10.16mm_Horizontal, B.Cu at (401.5, 213.2)
- added D38: 1N4001, Diode_THT:D_DO-41_SOD81_P10.16mm_Horizontal, B.Cu at (331.5, 246.5)
- added D39: 1N4001, Diode_THT:D_DO-41_SOD81_P10.16mm_Horizontal, B.Cu at (331.5, 76.5)
- added D40: 1N4001, Diode_THT:D_DO-41_SOD81_P10.16mm_Horizontal, B.Cu at (14.5, 88.7)
- added D41: 1N4001, Diode_THT:D_DO-41_SOD81_P10.16mm_Horizontal, B.Cu at (331.5, 156.5)
- added D42: 1N4001, Diode_THT:D_DO-41_SOD81_P10.16mm_Horizontal, B.Cu at (329.5, 195.4)
- added D43: 1N4001, Diode_THT:D_DO-41_SOD81_P10.16mm_Horizontal, B.Cu at (361.5, 76.5)
- added D44: 1N4001, Diode_THT:D_DO-41_SOD81_P10.16mm_Horizontal, B.Cu at (361.5, 116.5)
- added D45: 1N4001, Diode_THT:D_DO-41_SOD81_P10.16mm_Horizontal, B.Cu at (451.4, 206.5)
- added D46: 1N4001, Diode_THT:D_DO-41_SOD81_P10.16mm_Horizontal, B.Cu at (441.2, 154.8)
- added D47: 1N4001, Diode_THT:D_DO-41_SOD81_P10.16mm_Horizontal, B.Cu at (401.5, 76.5)
- added D48: 1N4001, Diode_THT:D_DO-41_SOD81_P10.16mm_Horizontal, B.Cu at (401.5, 116.5)
- added D49: 1N4001, Diode_THT:D_DO-41_SOD81_P10.16mm_Horizontal, B.Cu at (441.5, 196.5)
- added D50: 1N4001, Diode_THT:D_DO-41_SOD81_P10.16mm_Horizontal, B.Cu at (446.3, -3.50)
- added D51: 1N4001, Diode_THT:D_DO-41_SOD81_P10.16mm_Horizontal, B.Cu at (448.8, 76.0)
- added D52: 1N4001, Diode_THT:D_DO-41_SOD81_P10.16mm_Horizontal, B.Cu at (448.8, 114.1)
- added D53: 1N4001, Diode_THT:D_DO-41_SOD81_P10.16mm_Horizontal, B.Cu at (481.5, 156.5)
- added D54: 1N4001, Diode_THT:D_DO-41_SOD81_P10.16mm_Horizontal, B.Cu at (481.5, -3.50)
- added D55: 1N4001, Diode_THT:D_DO-41_SOD81_P10.16mm_Horizontal, B.Cu at (481.5, 73.5)
- added D56: 1N4001, Diode_THT:D_DO-41_SOD81_P10.16mm_Horizontal, B.Cu at (481.5, 114.1)
- added D57: 1N4001, Diode_THT:D_DO-41_SOD81_P10.16mm_Horizontal, B.Cu at (408.2, 154.8)
- added D58: 1N4001, Diode_THT:D_DO-41_SOD81_P10.16mm_Horizontal, B.Cu at (481.5, 196.5)
- added D59: 1N4001, Diode_THT:D_DO-41_SOD81_P10.16mm_Horizontal, B.Cu at (486.9, 248.7)
- added D60: 1N4001, Diode_THT:D_DO-41_SOD81_P10.16mm_Horizontal, B.Cu at (331.5, 126.8)
- added D61: 1N4001, Diode_THT:D_DO-41_SOD81_P10.16mm_Horizontal, B.Cu at (521.5, 196.5)
- added D62: 1N4001, Diode_THT:D_DO-41_SOD81_P10.16mm_Horizontal, B.Cu at (560.6, -3.50)
- added D63: 1N4001, Diode_THT:D_DO-41_SOD81_P10.16mm_Horizontal, B.Cu at (527.6, 76.0)
- added D64: 1N4001, Diode_THT:D_DO-41_SOD81_P10.16mm_Horizontal, B.Cu at (527.6, 116.5)
- added D65: 1N4001, Diode_THT:D_DO-41_SOD81_P10.16mm_Horizontal, B.Cu at (527.6, 154.8)
- added D66: 1N4001, Diode_THT:D_DO-41_SOD81_P10.16mm_Horizontal, B.Cu at (608.9, 27.8)
- added D67: 1N4001, Diode_THT:D_DO-41_SOD81_P10.16mm_Horizontal, B.Cu at (560.6, 48.1)
- added D68: 1N4001, Diode_THT:D_DO-41_SOD81_P10.16mm_Horizontal, B.Cu at (561.5, 116.7)
- added D69: 1N4001, Diode_THT:D_DO-41_SOD81_P10.16mm_Horizontal, B.Cu at (561.5, 156.5)
- added D7: 1N4001, Diode_THT:D_DO-41_SOD81_P10.16mm_Horizontal, B.Cu at (1.80, 195.4)
- added D70: 1N4001, Diode_THT:D_DO-41_SOD81_P10.16mm_Horizontal, B.Cu at (560.6, 195.4)
- added D71: 1N4001, Diode_THT:D_DO-41_SOD81_P10.16mm_Horizontal, B.Cu at (585.3, 203.0)
- added D72: 1N4001, Diode_THT:D_DO-41_SOD81_P10.16mm_Horizontal, B.Cu at (641.5, 1.42)
- added D73: 1N4001, Diode_THT:D_DO-41_SOD81_P10.16mm_Horizontal, B.Cu at (608.9, 45.5)
- added D74: 1N4001, Diode_THT:D_DO-41_SOD81_P10.16mm_Horizontal, B.Cu at (608.9, 114.1)
- added D75: 1N4001, Diode_THT:D_DO-41_SOD81_P10.16mm_Horizontal, B.Cu at (611.5, 156.5)
- added D76: 1N4001, Diode_THT:D_DO-41_SOD81_P10.16mm_Horizontal, B.Cu at (45.0, 167.5)
- added D77: 1N4001, Diode_THT:D_DO-41_SOD81_P10.16mm_Horizontal, B.Cu at (624.1, 137.0)
- added D78: 1N4001, Diode_THT:D_DO-41_SOD81_P10.16mm_Horizontal, B.Cu at (682.5, -5.26)
- added D79: 1N4001, Diode_THT:D_DO-41_SOD81_P10.16mm_Horizontal, B.Cu at (641.9, 73.5)
- added D8: 1N4001, Diode_THT:D_DO-41_SOD81_P10.16mm_Horizontal, B.Cu at (11.5, 243.7)
- added D80: 1N4001, Diode_THT:D_DO-41_SOD81_P10.16mm_Horizontal, B.Cu at (641.9, 114.1)
- added D81: 1N4001, Diode_THT:D_DO-41_SOD81_P10.16mm_Horizontal, B.Cu at (641.5, 166.5)
- added D82: 1N4001, Diode_THT:D_DO-41_SOD81_P10.16mm_Horizontal, B.Cu at (721.5, -3.50)
- added D83: 1N4001, Diode_THT:D_DO-41_SOD81_P10.16mm_Horizontal, B.Cu at (687.6, 45.5)
- added D84: 1N4001, Diode_THT:D_DO-41_SOD81_P10.16mm_Horizontal, B.Cu at (687.6, 114.1)
- added D85: 1N4001, Diode_THT:D_DO-41_SOD81_P10.16mm_Horizontal, B.Cu at (687.6, 157.3)
- added D86: 1N4001, Diode_THT:D_DO-41_SOD81_P10.16mm_Horizontal, B.Cu at (687.6, 192.9)
- added D87: 1N4001, Diode_THT:D_DO-41_SOD81_P10.16mm_Horizontal, B.Cu at (721.5, 116.5)
- added D88: 1N4001, Diode_THT:D_DO-41_SOD81_P10.16mm_Horizontal, B.Cu at (721.5, 156.5)
- added D89: 1N4001, Diode_THT:D_DO-41_SOD81_P10.16mm_Horizontal, B.Cu at (721.5, 192.9)
- added D9: 1N4001, Diode_THT:D_DO-41_SOD81_P10.16mm_Horizontal, B.Cu at (41.5, 45.5)
- added D90: 1N4001, Diode_THT:D_DO-41_SOD81_P10.16mm_Horizontal, B.Cu at (761.5, -3.50)
- added D91: 1N4001, Diode_THT:D_DO-41_SOD81_P10.16mm_Horizontal, B.Cu at (731.5, 46.5)
- added D92: 1N4001, Diode_THT:D_DO-41_SOD81_P10.16mm_Horizontal, B.Cu at (761.3, 192.9)
- added D93: 1N4001, Diode_THT:D_DO-41_SOD81_P10.16mm_Horizontal, B.Cu at (761.3, 213.2)
- added D94: 1N4001, Diode_THT:D_DO-41_SOD81_P10.16mm_Horizontal, B.Cu at (771.5, 46.5)
- added D95: 1N4001, Diode_THT:D_DO-41_SOD81_P10.16mm_Horizontal, B.Cu at (771.5, 116.5)
- added D96: 1N4001, Diode_THT:D_DO-41_SOD81_P10.16mm_Horizontal, B.Cu at (768.9, 157.3)
- added D97: 1N4001, Diode_THT:D_DO-41_SOD81_P10.16mm_Horizontal, B.Cu at (801.5, 45.5)
- added D98: 1N4001, Diode_THT:D_DO-41_SOD81_P10.16mm_Horizontal, B.Cu at (801.9, 116.7)
- added D99: 1N4001, Diode_THT:D_DO-41_SOD81_P10.16mm_Horizontal, B.Cu at (801.9, 157.3)
- added DELETE1: SW_SPST, Button_Switch_Keyboard:SW_Cherry_MX_1.00u_PCB, B.Cu at (241.5, 94.8)
- added D_1: SW_SPST, Button_Switch_Keyboard:SW_Cherry_MX_1.00u_PCB, B.Cu at (721.5, 136.5)
- added Down_Arrow1: SW_SPST, Button_Switch_Keyboard:SW_Cherry_MX_1.00u_PCB, B.Cu at (201.5, 221.6)
- added ELL_1: SW_SPST, Button_Switch_Keyboard:SW_Cherry_MX_1.00u_PCB, B.Cu at (481.5, 136.5)
- added END1: SW_SPST, Button_Switch_Keyboard:SW_Cherry_MX_1.00u_PCB, B.Cu at (201.5, 96.5)
- added ESC_1: SW_SPST, Button_Switch_Keyboard:SW_Cherry_MX_1.00u_PCB, B.Cu at (841.5, -23.5)
- added EYE_1: SW_SPST, Button_Switch_Keyboard:SW_Cherry_MX_1.00u_PCB, B.Cu at (521.5, 96.5)
- added E_1: SW_SPST, Button_Switch_Keyboard:SW_Cherry_MX_1.00u_PCB, B.Cu at (721.5, 96.5)
- added Enter1: SW_SPST, Button_Switch_Keyboard:SW_Cherry_MX_2.00u_PCB, B.Cu at (321.5, 136.5)
- added F1_1: SW_SPST, Button_Switch_Keyboard:SW_Cherry_MX_1.00u_PCB, B.Cu at (761.5, -23.5)
- added F2_1: SW_SPST, Button_Switch_Keyboard:SW_Cherry_MX_1.00u_PCB, B.Cu at (721.5, -23.5)
- added F3_1: SW_SPST, Button_Switch_Keyboard:SW_Cherry_MX_1.00u_PCB, B.Cu at (681.5, -23.5)
- added F4_1: SW_SPST, Button_Switch_Keyboard:SW_Cherry_MX_1.00u_PCB, B.Cu at (641.5, -23.5)
- added F5_1: SW_SPST, Button_Switch_Keyboard:SW_Cherry_MX_1.00u_PCB, B.Cu at (601.5, -23.5)
- added F6_1: SW_SPST, Button_Switch_Keyboard:SW_Cherry_MX_1.00u_PCB, B.Cu at (561.5, -23.5)
- added F7_1: SW_SPST, Button_Switch_Keyboard:SW_Cherry_MX_1.00u_PCB, B.Cu at (521.5, -23.5)
- added F8_1: SW_SPST, Button_Switch_Keyboard:SW_Cherry_MX_1.00u_PCB, B.Cu at (481.5, -23.5)
- added F9_1: SW_SPST, Button_Switch_Keyboard:SW_Cherry_MX_1.00u_PCB, B.Cu at (441.5, -23.5)
- added F_1: SW_SPST, Button_Switch_Keyboard:SW_Cherry_MX_1.00u_PCB, B.Cu at (681.5, 136.5)
- added G_1: SW_SPST, Button_Switch_Keyboard:SW_Cherry_MX_1.00u_PCB, B.Cu at (641.5, 136.5)
- added Greater_Than_1: SW_SPST, Button_Switch_Keyboard:SW_Cherry_MX_1.00u_PCB, B.Cu at (481.5, 176.5)
- added HOME1: SW_SPST, Button_Switch_Keyboard:SW_Cherry_MX_1.00u_PCB, B.Cu at (201.5, 56.5)
- added H_1: SW_SPST, Button_Switch_Keyboard:SW_Cherry_MX_1.00u_PCB, B.Cu at (601.5, 136.5)
- added INSERT1: SW_SPST, Button_Switch_Keyboard:SW_Cherry_MX_1.00u_PCB, B.Cu at (241.5, 56.5)
- added J_1: SW_SPST, Button_Switch_Keyboard:SW_Cherry_MX_1.00u_PCB, B.Cu at (561.5, 136.5)
- added KP_0_1: SW_SPST, Button_Switch_Keyboard:SW_Cherry_MX_2.00u_PCB, B.Cu at (1.50, 221.6)
- added KP_1_1: SW_SPST, Button_Switch_Keyboard:SW_Cherry_MX_1.00u_PCB, B.Cu at (81.5, 176.5)
- added KP_2_1: SW_SPST, Button_Switch_Keyboard:SW_Cherry_MX_1.00u_PCB, B.Cu at (41.5, 176.5)
- added KP_3_1: SW_SPST, Button_Switch_Keyboard:SW_Cherry_MX_1.00u_PCB, B.Cu at (1.50, 176.5)
- added KP_4_1: SW_SPST, Button_Switch_Keyboard:SW_Cherry_MX_1.00u_PCB, B.Cu at (81.5, 136.5)
- added KP_5_1: SW_SPST, Button_Switch_Keyboard:SW_Cherry_MX_1.00u_PCB, B.Cu at (41.5, 136.5)
- added KP_6_1: SW_SPST, Button_Switch_Keyboard:SW_Cherry_MX_1.00u_PCB, B.Cu at (1.50, 136.5)
- added KP_7_1: SW_SPST, Button_Switch_Keyboard:SW_Cherry_MX_1.00u_PCB, B.Cu at (81.5, 96.5)
- added KP_8_1: SW_SPST, Button_Switch_Keyboard:SW_Cherry_MX_1.00u_PCB, B.Cu at (41.5, 96.5)
- added KP_9_1: SW_SPST, Button_Switch_Keyboard:SW_Cherry_MX_1.00u_PCB, B.Cu at (1.50, 96.5)
- added KP_DOT_1: SW_SPST, Button_Switch_Keyboard:SW_Cherry_MX_1.00u_PCB, B.Cu at (51.5, 221.6)
- added KP_ENTER1: SW_SPST, Button_Switch_Keyboard:SW_Cherry_MX_2.00u_PCB, B.Cu at (-28.5, 176.5)
- added KP_NUM1: SW_SPST, Button_Switch_Keyboard:SW_Cherry_MX_1.00u_PCB, B.Cu at (81.5, 56.5)
- added K_1: SW_SPST, Button_Switch_Keyboard:SW_Cherry_MX_1.00u_PCB, B.Cu at (521.5, 136.5)
- added K_F10_1: SW_SPST, Button_Switch_Keyboard:SW_Cherry_MX_1.00u_PCB, B.Cu at (401.5, -23.5)
- added K_F11_1: SW_SPST, Button_Switch_Keyboard:SW_Cherry_MX_1.00u_PCB, B.Cu at (361.5, -23.5)
- added K_F12_1: SW_SPST, Button_Switch_Keyboard:SW_Cherry_MX_1.00u_PCB, B.Cu at (321.5, -23.5)
- added Left_Alt_1: SW_SPST, Button_Switch_Keyboard:SW_Cherry_MX_1.25u_PCB, B.Cu at (761.5, 221.6)
- added Left_Arrow1: SW_SPST, Button_Switch_Keyboard:SW_Cherry_MX_1.00u_PCB, B.Cu at (161.5, 221.6)
- added Left_Control_1: SW_SPST, Button_Switch_Keyboard:SW_Cherry_MX_1.25u_PCB, B.Cu at (841.5, 221.6)
- added Left_Shift_1: SW_SPST, Button_Switch_Keyboard:SW_Cherry_MX_2.00u_PCB, B.Cu at (841.5, 176.5)
- added Left_Shift_2: SW_SPST, Button_Switch_Keyboard:SW_Cherry_MX_2.00u_PCB, B.Cu at (881.5, 176.5)
- added Left_Win_1: SW_SPST, Button_Switch_Keyboard:SW_Cherry_MX_1.25u_PCB, B.Cu at (801.5, 221.6)
- added Less_Than_1: SW_SPST, Button_Switch_Keyboard:SW_Cherry_MX_1.00u_PCB, B.Cu at (521.5, 176.5)
- added M_1: SW_SPST, Button_Switch_Keyboard:SW_Cherry_MX_1.00u_PCB, B.Cu at (561.5, 176.5)
- added Minus1: SW_SPST, Button_Switch_Keyboard:SW_Cherry_MX_1.00u_PCB, B.Cu at (401.5, 56.5)
- added N_1: SW_SPST, Button_Switch_Keyboard:SW_Cherry_MX_1.00u_PCB, B.Cu at (601.5, 176.5)
- added O_1: SW_SPST, Button_Switch_Keyboard:SW_Cherry_MX_1.00u_PCB, B.Cu at (481.5, 96.5)
- added Open_Bracket_1: SW_SPST, Button_Switch_Keyboard:SW_Cherry_MX_1.00u_PCB, B.Cu at (401.5, 96.5)
- added PAGE_DOWN1: SW_SPST, Button_Switch_Keyboard:SW_Cherry_MX_1.00u_PCB, B.Cu at (161.5, 96.5)
- added PAGE_UP1: SW_SPST, Button_Switch_Keyboard:SW_Cherry_MX_1.00u_PCB, B.Cu at (161.5, 56.5)
- added P_1: SW_SPST, Button_Switch_Keyboard:SW_Cherry_MX_1.00u_PCB, B.Cu at (441.5, 96.5)
- added Pause1: SW_SPST, Button_Switch_Keyboard:SW_Cherry_MX_1.00u_PCB, B.Cu at (161.5, -23.5)
- added Print_Screen1: SW_SPST, Button_Switch_Keyboard:SW_Cherry_MX_1.00u_PCB, B.Cu at (241.5, -23.5)
- added Q_1: SW_SPST, Button_Switch_Keyboard:SW_Cherry_MX_1.00u_PCB, B.Cu at (801.5, 96.5)
- added Question_Mark_1: SW_SPST, Button_Switch_Keyboard:SW_Cherry_MX_1.00u_PCB, B.Cu at (441.5, 176.5)
- added R_1: SW_SPST, Button_Switch_Keyboard:SW_Cherry_MX_1.00u_PCB, B.Cu at (681.5, 96.5)
- added Right_Alt_1: SW_SPST, Button_Switch_Keyboard:SW_Cherry_MX_1.25u_PCB, B.Cu at (441.5, 221.6)
- added Right_Arrow1: SW_SPST, Button_Switch_Keyboard:SW_Cherry_MX_1.00u_PCB, B.Cu at (241.5, 221.6)
- added Right_Control1: SW_SPST, Button_Switch_Keyboard:SW_Cherry_MX_1.00u_PCB, B.Cu at (321.5, 221.6)
- added Right_Shift1: SW_SPST, Button_Switch_Keyboard:SW_Cherry_MX_2.00u_PCB, B.Cu at (321.5, 176.5)
- added Right_Windows1: SW_SPST, Button_Switch_Keyboard:SW_Cherry_MX_1.00u_PCB, B.Cu at (401.5, 221.6)
- added S_1: SW_SPST, Button_Switch_Keyboard:SW_Cherry_MX_1.00u_PCB, B.Cu at (761.5, 136.5)
- added Scroll_Lock1: SW_SPST, Button_Switch_Keyboard:SW_Cherry_MX_1.00u_PCB, B.Cu at (201.5, -23.5)
- added Semicolon_1: SW_SPST, Button_Switch_Keyboard:SW_Cherry_MX_1.00u_PCB, B.Cu at (401.5, 136.5)
- added Space_1: SW_SPST, Button_Switch_Keyboard:SW_Cherry_MX_6.25u_PCB, B.Cu at (579.0, 221.6)
- added TAB_1: SW_SPST, Button_Switch_Keyboard:SW_Cherry_MX_1.25u_PCB, B.Cu at (841.5, 96.5)
- added TILDE_1: SW_SPST, Button_Switch_Keyboard:SW_Cherry_MX_1.00u_PCB, B.Cu at (841.5, 56.5)
- added T_1: SW_SPST, Button_Switch_Keyboard:SW_Cherry_MX_1.00u_PCB, B.Cu at (641.5, 96.5)
- added U_1: SW_SPST, Button_Switch_Keyboard:SW_Cherry_MX_1.00u_PCB, B.Cu at (561.5, 96.5)
- added Up_Arrow1: SW_SPST, Button_Switch_Keyboard:SW_Cherry_MX_1.00u_PCB, B.Cu at (201.5, 176.5)
- added V_1: SW_SPST, Button_Switch_Keyboard:SW_Cherry_MX_1.00u_PCB, B.Cu at (681.5, 176.5)
- added W_1: SW_SPST, Button_Switch_Keyboard:SW_Cherry_MX_1.00u_PCB, B.Cu at (761.5, 96.5)
- added X_1: SW_SPST, Button_Switch_Keyboard:SW_Cherry_MX_1.00u_PCB, B.Cu at (761.5, 176.5)
- added Y_1: SW_SPST, Button_Switch_Keyboard:SW_Cherry_MX_1.00u_PCB, B.Cu at (601.2, 96.5)
- added Z_1: SW_SPST, Button_Switch_Keyboard:SW_Cherry_MX_1.00u_PCB, B.Cu at (801.5, 176.5)
- added Zero_1: SW_SPST, Button_Switch_Keyboard:SW_Cherry_MX_1.00u_PCB, B.Cu at (441.5, 56.5)
- D1, D2, D3, D4, D5, D6, KP_MINUS1, KP_SLASH1, KP_STAR1, header1: moved to B.Cu
- KP_PLUS1: footprint Button_Switch_Keyboard:SW_Cherry_MX_1.00u_PCB -> Button_Switch_Keyboard:SW_Cherry_MX_2.00u_PCB; moved to B.Cu
- moved D5 194.9 mm to (1.80, 116.7)
- moved D3 186.5 mm to (-18.5, 186.5), turned to 90 degrees
- moved D2 175.9 mm to (-18.5, 126.5), turned to 90 degrees
- moved D1 166.2 mm to (-48.5, 56.5)
- moved D4 151.7 mm to (1.50, 35.4)
- moved KP_MINUS1 146.4 mm to (-36.3, 56.5), turned to 180 degrees
- moved D6 141.6 mm to (1.50, 156.5), turned to -90 degrees
- moved KP_PLUS1 140.2 mm to (-28.5, 116.5), turned to 90 degrees
- moved header1 134.8 mm to (-31.8, -16.9)
- moved KP_STAR1 128.7 mm to (1.50, 56.5), turned to 180 degrees
- moved KP_SLASH1 107.7 mm to (41.5, 56.5), turned to 180 degrees
Connections:
- D1 pad 1: Net-(KP_PLUS1-Pad1) -> Net-(KP_MINUS1-Pad1)
- D1 pad 2: Net-(header1-Pad19) -> Tag2
- D2 pad 2: Net-(header1-Pad19) -> Tag14
- D3 pad 1: Net-(KP_MINUS1-Pad1) -> Net-(KP_ENTER1-Pad2)
- D3 pad 2: Net-(header1-Pad22) -> Tag21
- D4 pad 2: Net-(header1-Pad19) -> Tag19
- D5 pad 1: Net-(KP_SLASH1-Pad1) -> Net-(D5-Pad1)
- D5 pad 2: Net-(header1-Pad19) -> Tag14
- D6 pad 2: Net-(header1-Pad19) -> Tag13
- KP_MINUS1 pad 2: Net-(header1-Pad19) -> Tag15
- KP_PLUS1 pad 1: Net-(KP_PLUS1-Pad1) -> Tag4
- KP_PLUS1 pad 2: Net-(header1-Pad26) -> Net-(D2-Pad1)
- KP_SLASH1 pad 1: Net-(KP_SLASH1-Pad1) -> Net-(D9-Pad1)
- KP_SLASH1 pad 2: Net-(KP_8-Pad2) -> Tag16
- KP_STAR1 pad 2: Net-(KP_STAR1-Pad2) -> Tag15
- header1 pad 1: unconnected-(header1-Pad1) -> Tag7
- header1 pad 10: unconnected-(header1-Pad10) -> Tag6
- header1 pad 11: unconnected-(header1-Pad11) -> Tag7
- header1 pad 12: unconnected-(header1-Pad12) -> Tag5
- header1 pad 13: unconnected-(header1-Pad13) -> Tag16
- header1 pad 14: unconnected-(header1-Pad14) -> Tag6
- header1 pad 15: unconnected-(header1-Pad15) -> Tag18
- header1 pad 16: unconnected-(header1-Pad16) -> Tag20
- header1 pad 17: unconnected-(header1-Pad17) -> Tag21
- header1 pad 18: unconnected-(header1-Pad18) -> Tag13
- header1 pad 19: Net-(header1-Pad19) -> Tag14
- header1 pad 2: unconnected-(header1-Pad2) -> Tag24
- header1 pad 20: unconnected-(header1-Pad20) -> Tag15
- header1 pad 21: Net-(header1-Pad19) -> Tag19
- header1 pad 22: Net-(header1-Pad22) -> Tag2
- header1 pad 23: unconnected-(header1-Pad23) -> Tag3
- header1 pad 24: unconnected-(header1-Pad24) -> Tag23
- header1 pad 25: unconnected-(header1-Pad25) -> Tag1
- header1 pad 26: Net-(header1-Pad26) -> Tag4
- header1 pad 3: unconnected-(header1-Pad3) -> Tag22
- header1 pad 4: unconnected-(header1-Pad4) -> Tag25
- header1 pad 5: unconnected-(header1-Pad5) -> Tag10
- header1 pad 6: unconnected-(header1-Pad6) -> Tag26
- header1 pad 7: unconnected-(header1-Pad7) -> Tag12
- header1 pad 8: unconnected-(header1-Pad8) -> Tag11
- header1 pad 9: unconnected-(header1-Pad9) -> Tag17
