File: das keyboard/das keyboard.kicad_sch (KiCad schematic)
At the start: 211 parts

Commit message: updates to the pcb
Parts:
- added D71, D87, D93: 1N4001, Diode_THT:D_DO-41_SOD81_P10.16mm_Horizontal, symbol Diode:1N4001
- gave numbers to parts that had none: 68
- renumbered Enter to Enter1, Minus to Minus1, Right_Shift to Right_Shift1
Connections:
- net Tag8 is gone; now on net Tag24: header1.2 (Pin_2)
- net Tag12: no longer D106.2 (A), D108.2 (A), F3_1.2 (B), F4_1.2 (B), Left_Win_1.2 (B), header1.24 (Pin_24)
- net Tag14: now also D84.2 (A), D87.2 (A); no longer E_1.1 (A)
- net Tag18: now also Down_Arrow1.1 (A), Space_1.1 (A)
- net Tag5: no longer Print_Screen1.1 (A), Right_Alt_1.2 (B), Scroll_Lock1.1 (A)
- net Tag7: now also +=1.2 (B), 8_1.1 (A), Close_Bracket1.2 (B), F6_1.2 (B), K_1.1 (A), header1.1 (Pin_1)
- net at D17.2 (A), D25.2 (A), D46.2 (A)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: now also D71.2 (A), D93.2 (A)
- net Tag21: now reaches D37.2 (A), D40.2 (A), D42.2 (A), D53.2 (A), D57.2 (A), D65.2 (A), D69.2 (A), D85.2 (A), D88.2 (A)
- net Tag21: now also D12.2 (A), D16.2 (A), D3.2 (A), D7.2 (A), header1.17 (Pin_17)
- net Tag22: now reaches 9_1.2 (B), D64.2 (A), D68.2 (A), ELL_1.2 (B), F7_1.1 (A), F8_1.2 (B), O_1.2 (B)
- net Tag22: now also header1.3 (Pin_3)
- net Tag26: now reaches 3_1.1 (A), C_1.2 (B), D_1.2 (B), E_1.2 (B)
- net Tag26: now also F2_1.2 (B), F3_1.2 (B), F4_1.2 (B), header1.6 (Pin_6); no longer D84.2 (A)
- net at D101.1 (K), D102.1 (K), Left_Shift_2.1 (A): no longer D103.2 (A)
- net Tag25: now reaches 6_1.1 (A), 7_1.2 (B), H_1.1 (A), J_1.2 (B), M_1.2 (B), N_1.1 (A), U_1.2 (B), Y_1.1 (A)
- net Tag25: now also header1.4 (Pin_4)
- net at D61.1 (K), Less_Than_1.1 (A): no longer K_1.1 (A)
- net at Left_Alt_1.1 (A): now also D93.1 (K)
- net Tag24: now reaches Left_Alt_1.2 (B)
- net Tag24: now also Print_Screen1.1 (A), Right_Alt_1.2 (B), Scroll_Lock1.1 (A)
- net at D74.2 (A), D78.2 (A), D80.2 (A): no longer D82.2 (A), D90.2 (A)
- net at Space_1.2 (B): now also D71.1 (K)
- net at D101.2 (A), D104.2 (A), D107.2 (A): now also D103.2 (A)
- new net: D106.2 (A), D108.2 (A)
- new net: D87.1 (K), E_1.1 (A)
- new net: D82.2 (A), D90.2 (A)
- new net Tag23: Left_Win_1.2 (B), header1.24 (Pin_24)
- now unconnected: EYE_1.1 (A)
Other:
- moved on the sheet: +=1, 1_1, 2_1, 3_1, 4_1, 5_1, 6_1, 7_1, 8_1, 9_1, APPS1, A_1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
